File: hw/sch_pcb/SPIEX01.kicad_pcb (KiCad board)
At the start: 2 copper layers, 50.3 x 50.3 mm, 20 parts, among them J1 PWR, P1 SPI-IN, P10 CONN_01X01, P11 CONN_01X01, P12 CONN_01X01, P13 CONN_01X01, P2 SPI3, P3 SPI0, P4 SPI4, P5 SPI1, P6 SPI5, P7 SPI2, P8 SPI6, U1 74HC00, U2 74HC164, U3 74HC125

Commit message: Uptade PCB file to KiCADv7.
Other:
- net class Default removed
- net class III removed
